File: Schematic & Layout/projektorosch.kicad_pcb (KiCad board)
At the start: 2 copper layers, 92.3 x 67.8 mm, 24 parts, among them J1 Barrel_Jack_Switch, J2 Conn_01x03, J3 RJ12, U1 ATtiny214-SS, U2 MAX232

Commit message: fixes
Parts:
- added H1: MountingHole, MountingHole:MountingHole_2.7mm, F.Cu at (195.0, 132.0)
- added H2: MountingHole, MountingHole:MountingHole_2.7mm, F.Cu at (112.0, 73.0)
- added H3: MountingHole, MountingHole:MountingHole_2.7mm, F.Cu at (195.0, 73.0)
- added H4: MountingHole, MountingHole:MountingHole_2.7mm, F.Cu at (112.0, 132.0)
- J1, U2: moved to B.Cu
- J3: footprint Connector_RJ:RJ12_Amphenol_54601 -> Connector_RJ:rj12_Sajat; moved to B.Cu
- moved C8 21.3 mm to (144.1, 109.4), turned to -90 degrees
- moved C6 16.9 mm to (144.6, 102.9)
- moved C5 14.7 mm to (133.2, 118.3), turned to 180 degrees
- moved J3 14.4 mm to (193.9, 119.6), turned to -90 degrees
- moved C4 14.2 mm to (147.4, 109.3)
- moved C7 9.86 mm to (147.3, 94.0)
- moved R10 6.54 mm to (140.3, 118.3)
- moved U2 5.16 mm to (152.4, 111.8), turned to 0 degrees
- moved J1 3.90 mm to (186.0, 83.6)
- moved C3 2.56 mm to (173.9, 81.3)
- moved D1 2.56 mm to (176.8, 81.3)
- moved F1 2.56 mm to (180.8, 81.4)
- moved C1 1.77 mm to (133.2, 113.7)
- moved C2 0.33 mm to (133.5, 109.4)
Connections:
- J3 pad 2: TX -> unconnected-(J3-Pad2)
- J3 pad 3: RX -> unconnected-(J3-Pad3)
- J3 pad 5: unconnected-(J3-Pad5) -> TX
- J3 pad 6: unconnected-(J3-Pad6) -> RX
- U1 pad 11: BTN3 -> unconnected-(U1-Pad11)
- U1 pad 12: BTN3LED -> BTN3
- U1 pad 13: unconnected-(U1-Pad13) -> BTN3LED
- U1 pad 3: BTN4 -> BTN2LED
- U1 pad 4: BTN2LED -> BTN4
Routing:
- net BTN4: track 36.5 -> 52.1 mm
- net Net-(BTN4-Pad3): track 35.1 -> 20.7 mm
- net VCC: track 176.4 -> 190.6 mm
- net TX: track 45.2 -> 33.8 mm
- net Net-(C8-Pad1): track 20.7 -> 9.42 mm
- net TXD: track 14.6 -> 25.4 mm
- net RXD: track 15.1 -> 25.9 mm
- net BTN4LED: track 7.44 -> 15.6 mm
- net RX: track 43.2 -> 37.3 mm
- net Net-(C6-Pad2): track 4.26 -> 7.84 mm
- net Net-(C6-Pad1): track 4.28 -> 7.84 mm
- net Net-(C7-Pad2): track 10.1 -> 6.59 mm
- net BTN3LED: track 9.12 -> 7.47 mm
- net BTN2LED: track 34.1 -> 35.5 mm
- net Net-(F1-Pad2): track 6.26 -> 5.39 mm
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
Commit message: final
Parts:
- BTN1, BTN2, BTN3, BTN4, J2: moved to B.Cu
- moved C5 30.9 mm to (163.0, 110.2), turned to 90 degrees
- moved C8 13.2 mm to (156.0, 115.0), turned to 0 degrees
- moved R9 5.27 mm to (126.4, 105.8), turned to 0 degrees
- moved C7 3.90 mm to (149.5, 97.2)
- moved C1 1.67 mm to (133.0, 112.0)
- turned BTN3 to 0 degrees
- turned J2 to 0 degrees
Connections:
- BTN1 pad 1: GND -> BTN1
- BTN1 pad 2: BTN1 -> GND
- BTN2 pad 1: GND -> BTN2
- BTN2 pad 2: BTN2 -> GND
- BTN3 pad 1: GND -> BTN3
- BTN3 pad 2: BTN3 -> GND
Routing:
- net VCC: track 190.6 -> 219.9 mm
- net BTN3: track 25.6 -> 35.2 mm
- net Net-(BTN3-Pad3): track 11.9 -> 20.3 mm
- net BTN4: track 52.1 -> 43.9 mm
- net RXD: track 25.9 -> 33.5 mm
- net TXD: track 25.4 -> 32.4 mm
- net BTN3LED: track 7.47 -> 3.14 mm
- net Net-(C7-Pad2): track 6.59 -> 2.55 mm
- net BTN1: track 22.2 -> 25.2 mm
- net Net-(C8-Pad1): track 9.42 -> 7.41 mm
- net BTN2: track 42.0 -> 43.1 mm
- net BTN4LED: track 15.6 -> 14.6 mm
Other:
- board text added: "2022.03.29. by Dvid"
- board text added: "ProjektoroSCH"

Commit message: normal buttons
Parts:
- removed BTN1, BTN2, BTN3, BTN4: LEDBTN, ledbtn_footprint:LBTN
- removed R10, R2, R5, R9: 220R, Resistor_SMD:R_0805_2012Metric_Pad1.20x1.40mm_HandSolder
- added U3: BTN, Button_Switch_THT:SW_PUSH_6mm_H5mm, F.Cu at (160.0, 80.0)
- added U4: BTN, Button_Switch_THT:SW_PUSH_6mm_H5mm, F.Cu at (121.0, 80.0)
- added U5: BTN, Button_Switch_THT:SW_PUSH_6mm_H5mm, F.Cu at (160.0, 120.0)
- added U6: BTN, Button_Switch_THT:SW_PUSH_6mm_H5mm, F.Cu at (121.0, 120.0)
Connections:
- U1 pad 13: BTN3LED -> unconnected-(U1-Pad13)
- U1 pad 2: BTN4LED -> unconnected-(U1-Pad2)
- U1 pad 3: BTN2LED -> unconnected-(U1-Pad3)
- U1 pad 9: BTN1LED -> unconnected-(U1-Pad9)
Routing:
- net BTN2LED: track 35.4 -> 0.00 mm
- net Net-(BTN4-Pad3): track 20.7 -> 0.00 mm
- net Net-(BTN3-Pad3): track 20.3 -> 0.00 mm
- net Net-(BTN1-Pad3): track 18.3 -> 0.00 mm
- net BTN4LED: track 14.6 -> 0.00 mm
- net BTN1: track 25.2 -> 32.0 mm
- net BTN1LED: track 6.76 -> 0.00 mm
- net BTN3: track 35.2 -> 30.0 mm
- net Net-(BTN2-Pad3): track 4.53 -> 0.00 mm
- net BTN3LED: track 3.14 -> 0.00 mm
- net BTN2: track 43.1 -> 45.1 mm
- net BTN4: track 43.9 -> 45.4 mm
