File: Schematic & Layout/projektorosch.kicad_sch (KiCad schematic)
At the start: 28 parts, among them J1 Barrel_Jack_Switch, J2 Conn_01x03, J3 RJ12, U1 ATtiny214-SS, U2 MAX232

Commit message: final
Connections:
- net BTN1: now also BTN1.1; no longer BTN1.2
- net BTN2: now also BTN2.1; no longer BTN2.2
- net BTN3: now also BTN3.1; no longer BTN3.2
- net GND: now also BTN1.2, BTN2.2, BTN3.2; no longer BTN1.1, BTN2.1, BTN3.1
Changed lines of the file:
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@@
-    (stroke (width 0) (type default) (color 0 0 0 0))
-  )
-  (wire (pts (xy 152.908 174.498) (xy 150.368 174.498))
     (stroke (width 0) (type default) (color 0 0 0 0))
   )
@@
     (stroke (width 0) (type default) (color 0 0 0 0))
   )
-  (wire (pts (xy 85.09 134.874) (xy 85.09 136.525))
-    (stroke (width 0) (type default) (color 0 0 0 0))
-  )
   (wire (pts (xy 199.39 62.738) (xy 199.39 65.278))
     (stroke (width 0) (type default) (color 0 0 0 0))
@@
     (stroke (width 0) (type default) (color 0 0 0 0))
   )
-  (wire (pts (xy 150.622 133.858) (xy 148.082 133.858))
-    (stroke (width 0) (type default) (color 0 0 0 0))
-  )
   (wire (pts (xy 237.49 98.298) (xy 236.22 98.298))
     (stroke (width 0) (type default) (color 0 0 0 0))
@@
     (stroke (width 0) (type default) (color 0 0 0 0))
   )
-  (wire (pts (xy 89.154 134.874) (xy 85.09 134.874))
-    (stroke (width 0) (type default) (color 0 0 0 0))
-  )
   (wire (pts (xy 106.045 69.85) (xy 107.315 69.85))
     (stroke (width 0) (type default) (color 0 0 0 0))
@@
     (stroke (width 0) (type default) (color 0 0 0 0))
   )
-  (wire (pts (xy 100.584 134.62) (xy 105.41 134.62))
-    (stroke (width 0) (type default) (color 0 0 0 0))
-  )
   (wire (pts (xy 237.49 107.95) (xy 237.49 138.938))
     (stroke (width 0) (type default) (color 0 0 0 0))
@@
     (stroke (width 0) (type default) (color 0 0 0 0))
   )
-  (wire (pts (xy 133.858 174.752) (xy 138.938 174.752))
-    (stroke (width 0) (type default) (color 0 0 0 0))
-  )
   (wire (pts (xy 37.465 171.45) (xy 42.545 171.45))
     (stroke (width 0) (type default) (color 0 0 0 0))
@@
   )
   (wire (pts (xy 233.68 105.918) (xy 237.49 105.918))
-    (stroke (width 0) (type default) (color 0 0 0 0))
-  )
-  (wire (pts (xy 103.632 173.736) (xy 101.092 173.736))
     (stroke (width 0) (type default) (color 0 0 0 0))
   )
@@
     )
   )
-  (global_label "BTN4" (shape input) (at 152.908 174.498 0) (fields_autoplaced)
-    (effects (font (size 1.27 1.27)) (justify left))
-    (property "Intersheet References" "${INTERSHEET_REFS}" (id 0) (at 160.0987 174.4186 0)
-      (effects (font (size 1.27 1.27)) (justify left) hide)
-    )
-  )
-  (global_label "BTN2" (shape input) (at 103.632 173.736 0) (fields_autoplaced)
-    (effects (font (size 1.27 1.27)) (justify left))
-    (property "Intersheet References" "${INTERSHEET_REFS}" (id 0) (at 110.8227 173.6566 0)
-      (effects (font (size 1.27 1.27)) (justify left) hide)
+  (global_label "BTN4" (shape input) (at 150.368 174.498 0) (fields_autoplaced)
+    (effects (font (size 1.27 1.27)) (justify left))
+    (property "Intersheet References" "${INTERSHEET_REFS}" (id 0) (at 157.5587 174.4186 0)
+      (effects (font (size 1.27 1.27)) (justify left) hide)
+    )
+  )
+  (global_label "BTN2" (shape input) (at 89.662 173.99 180) (fields_autoplaced)
+    (effects (font (size 1.27 1.27)) (justify right))
+    (property "Intersheet References" "${INTERSHEET_REFS}" (id 0) (at 82.4713 174.0694 0)
+      (effects (font (size 1.27 1.27)) (justify right) hide)
     )
   )
@@
     )
   )
-  (global_label "BTN3" (shape input) (at 150.622 133.858 0) (fields_autoplaced)
-    (effects (font (size 1.27 1.27)) (justify left))
-    (property "Intersheet References" "${INTERSHEET_REFS}" (id 0) (at 157.8127 133.7786 0)
-      (effects (font (size 1.27 1.27)) (justify left) hide)
-    )
-  )
-  (global_label "BTN1" (shape input) (at 105.41 134.62 0) (fields_autoplaced)
-    (effects (font (size 1.27 1.27)) (justify left))
-    (property "Intersheet References" "${INTERSHEET_REFS}" (id 0) (at 112.6007 134.5406 0)
-      (effects (font (size 1.27 1.27)) (justify left) hide)
+  (global_label "BTN3" (shape input) (at 136.652 134.112 180) (fields_autoplaced)
+    (effects (font (size 1.27 1.27)) (justify right))
+    (property "Intersheet References" "${INTERSHEET_REFS}" (id 0) (at 129.4613 134.1914 0)
+      (effects (font (size 1.27 1.27)) (justify right) hide)
+    )
+  )
+  (global_label "BTN1" (shape input) (at 89.154 134.874 180) (fields_autoplaced)
+    (effects (font (size 1.27 1.27)) (justify right))
+    (property "Intersheet References" "${INTERSHEET_REFS}" (id 0) (at 81.9633 134.9534 0)
+      (effects (font (size 1.27 1.27)) (justify right) hide)
     )
   )
@@
     )
   )
-  (symbol (lib_id "power:GND") (at 136.652 134.112 0) (mirror y) (unit 1)
-    (in_bom yes) (on_board yes) (fields_autoplaced)
-    (property "Reference" "#PWR0101" (id 0) (at 136.652 140.462 0)
-      (effects (font (size 1.27 1.27)) hide)
-    )
-    (property "Value" "GND" (id 1) (at 136.652 138.557 0))
-    (property "Footprint" "" (id 2) (at 136.652 134.112 0)
-      (effects (font (size 1.27 1.27)) hide)
-    )
-    (property "Datasheet" "" (id 3) (at 136.652 134.112 0)
+  (symbol (lib_id "power:GND") (at 148.082 133.858 0) (mirror y) (unit 1)
+    (in_bom yes) (on_board yes) (fields_autoplaced)
+    (property "Reference" "#PWR0101" (id 0) (at 148.082 140.208 0)
+      (effects (font (size 1.27 1.27)) hide)
+    )
+    (property "Value" "GND" (id 1) (at 148.082 138.303 0))
+    (property "Footprint" "" (id 2) (at 148.082 133.858 0)
+      (effects (font (size 1.27 1.27)) hide)
+    )
+    (property "Datasheet" "" (id 3) (at 148.082 133.858 0)
       (effects (font (size 1.27 1.27)) hide)
     )
@@
     (pin "1")
   )
-  (symbol (lib_id "power:GND") (at 133.858 174.752 0) (mirror y) (unit 1)
-    (in_bom yes) (on_board yes) (fields_autoplaced)
-    (property "Reference" "#PWR0102" (id 0) (at 133.858 181.102 0)
-      (effects (font (size 1.27 1.27)) hide)
-    )
-    (property "Value" "GND" (id 1) (at 133.858 179.197 0))
-    (property "Footprint" "" (id 2) (at 133.858 174.752 0)
-      (effects (font (size 1.27 1.27)) hide)
-    )
-    (property "Datasheet" "" (id 3) (at 133.858 174.752 0)
+  (symbol (lib_id "power:GND") (at 138.938 174.752 0) (mirror y) (unit 1)
+    (in_bom yes) (on_board yes) (fields_autoplaced)
+    (property "Reference" "#PWR0102" (id 0) (at 138.938 181.102 0)
+      (effects (font (size 1.27 1.27)) hide)
+    )
+    (property "Value" "GND" (id 1) (at 138.938 179.197 0))
+    (property "Footprint" "" (id 2) (at 138.938 174.752 0)
+      (effects (font (size 1.27 1.27)) hide)
+    )
+    (property "Datasheet" "" (id 3) (at 138.938 174.752 0)
       (effects (font (size 1.27 1.27)) hide)
     )
@@
     )
   )
-  (symbol (lib_id "power:GND") (at 89.662 173.99 0) (unit 1)
-    (in_bom yes) (on_board yes) (fields_autoplaced)
-    (property "Reference" "#PWR012" (id 0) (at 89.662 180.34 0)
-      (effects (font (size 1.27 1.27)) hide)
-    )
-    (property "Value" "GND" (id 1) (at 89.662 179.07 0))
-    (property "Footprint" "" (id 2) (at 89.662 173.99 0)
-      (effects (font (size 1.27 1.27)) hide)
-    )
-    (property "Datasheet" "" (id 3) (at 89.662 173.99 0)
+  (symbol (lib_id "power:GND") (at 101.092 173.736 0) (unit 1)
+    (in_bom yes) (on_board yes) (fields_autoplaced)
+    (property "Reference" "#PWR012" (id 0) (at 101.092 180.086 0)
+      (effects (font (size 1.27 1.27)) hide)
+    )
+    (property "Value" "GND" (id 1) (at 101.092 178.816 0))
+    (property "Footprint" "" (id 2) (at 101.092 173.736 0)
+      (effects (font (size 1.27 1.27)) hide)
+    )
+    (property "Datasheet" "" (id 3) (at 101.092 173.736 0)
       (effects (font (size 1.27 1.27)) hide)
     )
@@
     (pin "1")
   )
-  (symbol (lib_id "power:GND") (at 85.09 136.525 0) (mirror y) (unit 1)
-    (in_bom yes) (on_board yes) (fields_autoplaced)
-    (property "Reference" "#PWR011" (id 0) (at 85.09 142.875 0)
-      (effects (font (size 1.27 1.27)) hide)
-    )
-    (property "Value" "GND" (id 1) (at 85.09 140.97 0))
-    (property "Footprint" "" (id 2) (at 85.09 136.525 0)
-      (effects (font (size 1.27 1.27)) hide)
-    )
-    (property "Datasheet" "" (id 3) (at 85.09 136.525 0)
-      (effects (font (size 1.27 1.27)) hide)
-    )
+  (symbol (lib_id "power:GND") (at 100.584 134.62 0) (mirror y) (unit 1)
+    (in_bom yes) (on_board yes) (fields_autoplaced)
+    (property "Reference" "#PWR011" (id 0) (at 100.584 140.97 0)
+      (effects (font (size 1.27 1.27)) hide)
+    )
+    (property "Value" "GND" (id 1) (at 100.584 139.065 0))
+    (property "Footprint" "" (id 2) (at 100.584 134.62 0)
+      (effects (font (size 1.27 1.27)) hide)
+    )
+    (property "Datasheet" "" (id 3) (at 100.584 134.62 0)
+      (effects (font (size 1.27 1.27)) hide)
+    )

Commit message: normal buttons
Parts:
- removed BTN1, BTN2, BTN3, BTN4: LEDBTN, ledbtn_footprint:LBTN, symbol projektorosch:LEDBTN
- removed R10, R2, R5, R9: 220R, Resistor_SMD:R_0805_2012Metric_Pad1.20x1.40mm_HandSolder, symbol Device:R
- added U3, U4, U5, U6: BTN, Button_Switch_THT:SW_PUSH_6mm_H5mm, symbol projektorosch:BTN
Connections:
- net BTN1: now also U4.1
- net BTN2: now also U3.1
- net BTN3: now also U6.1
- net BTN4: now also U5.1
- net GND: now also U3.2, U4.2, U5.2, U6.2
- net BTN1LED: no longer names the net of U1.9 (PB0)
- net BTN2LED: no longer names the net of U1.3 (PA5)
- net BTN3LED: no longer names the net of U1.13 (PA3)
- net BTN4LED: no longer names the net of U1.2 (PA4)
